Commit message: Add a safety layer: people and obstacle detection, tool hold, reroute
- safety_monitor node per robot sits between the planner (cmd_vel_nav)
  and the wheels (cmd_vel): lidar clustering and tracking in the
  wheel-odometry frame, ground hits dropped using the survey DEM and
  IMU tilt, speed-and-separation zones for people and static objects,
  crossing prediction, latched e-stop, watchdog, geofence.
- Tool hold: a person within 2 m of the auger or duckbill freezes the
  mechanisms; fs::AugerSoil gains hold/resume so a bore pauses mid-hole.
- Jaal waits for people, goes round static objects on a free side,
  skips a spot an obstacle covers; Pahadi waits and calls the operator;
  Katar guards the boom strip.
- Rear lidar on Jaal, boom-side lidar on Katar, Pahadi lidar on by
  default; SafetyStatus message; RViz safety markers.
- pedestrians node, person and crate models: launch people:=all to run
  crossing, tool, standing-person and crate scenarios.
- Unit tests for the safety logic and the launch wiring.

Co-Authored-By: Claude Opus 5.5 <noreply@anthropic.com>

File: ros2_ws/src/fs_description/urdf/common.xacro (robot description, xacro)
@@ -118,13 +118,14 @@
   </xacro:macro>
   <!-- Planar safety lidar. Needs rendering (gpu_lidar); off with lidar:=false. -->
-  <xacro:macro name="lidar2d" params="ns parent xyz fov:=4.71 samples:=540 max_range:=20.0">
-    <joint name="lidar_joint" type="fixed"><parent link="${parent}"/><child link="lidar_link"/><origin xyz="${xyz}"/></joint>
-    <link name="lidar_link">
+  <!-- Planar lidar. name/topic let one robot carry several (Jaal front and rear). -->
+  <xacro:macro name="lidar2d" params="ns parent xyz rpy:='0 0 0' name:=lidar topic:=scan fov:=4.71 samples:=540 max_range:=20.0">
+    <joint name="${name}_joint" type="fixed"><parent link="${parent}"/><child link="${name}_link"/><origin xyz="${xyz}" rpy="${rpy}"/></joint>
+    <link name="${name}_link">
       <visual><geometry><cylinder radius="0.05" length="0.07"/></geometry><material name="fs_graphite"/></visual>
     </link>
-    <gazebo reference="lidar_link">
-      <sensor name="lidar" type="gpu_lidar">
-        <always_on>1</always_on><update_rate>10</update_rate><topic>/model/${ns}/scan</topic>
-        <gz_frame_id>${ns}/lidar_link</gz_frame_id>
+    <gazebo reference="${name}_link">
+      <sensor name="${name}" type="gpu_lidar">
+        <always_on>1</always_on><update_rate>10</update_rate><topic>/model/${ns}/${topic}</topic>
+        <gz_frame_id>${ns}/${name}_link</gz_frame_id>
         <lidar>
           <scan><horizontal><samples>${samples}</samples><resolution>1</resolution>

File: ros2_ws/src/fs_description/urdf/jaal.urdf.xacro (robot description, xacro)
@@ -111,4 +111,6 @@
   <xacro:if value="$(arg lidar)">
     <xacro:lidar2d ns="${ns}" parent="base_link" xyz="1.52 0 -0.08"/>  <!-- 0.30 m above ground: sees stumps -->
+    <!-- rear: the planting head works at the back, where people walk up to it -->
+    <xacro:lidar2d ns="${ns}" parent="base_link" xyz="-1.52 0 -0.08" rpy="0 0 3.14159" name="lidar_rear" topic="scan_rear"/>
   </xacro:if>
   <xacro:if value="$(arg inspect_cam)">

File: ros2_ws/src/fs_description/urdf/katar.urdf.xacro (robot description, xacro)
@@ -100,4 +100,6 @@
   <xacro:auger_head robot="${R}" parent="turret_link" xyz="0.2 0 -0.06" length="0.95" stroke="1.3"/>
   <xacro:duckbill_head robot="${R}" parent="turret_link" xyz="-0.2 0 -0.06" stroke="1.6" tamp_xyz="-0.2 0 -0.20" tamp_stroke="1.6"/>
+  <!-- boom-side lidar, 0.3 m above ground, watching the strip the boom works in -->
+  <xacro:lidar2d ns="${ns}" parent="trailer_link" xyz="-1.5 1.08 -0.2" rpy="0 0 1.5708"/>
   <xacro:if value="$(arg inspect_cam)">
     <!-- rides on the boom carriage so the head stays in frame -->

File: ros2_ws/src/fs_description/urdf/pahadi.urdf.xacro (robot description, xacro)
@@ -12,5 +12,5 @@
   <xacro:arg name="ns" default="pahadi"/>
   <xacro:arg name="soil_map" default=""/>
-  <xacro:arg name="lidar" default="false"/>
+  <xacro:arg name="lidar" default="true"/>
   <xacro:arg name="gnss_sigma" default="0.02"/>
   <xacro:property name="ns" value="$(arg ns)"/>

Commit message: Ground the models in CAD physics, deepen the soil model, and add a hardware bringup
- Feed masts and carriages carry the auger, duckbill and tamp ring on all three robots, so no tool
  hangs in mid-air; amendment hoppers with screw feeders; Katar's 1.45 m deep-auger kit
- Link inertials integrated from the CAD solids and loaded into the URDF at spawn; realistic
  wheel torque limits per robot
- Physics audit (ros2 run fs_bringup physics_audit): inertia, mass and CoM, articulated contact
  loads, tip angles, sinkage, gradeability (dry and monsoon), auger reaction, arm torques
- Soil: moisture-dependent strength, a shared multi-pass rut map, and auger-hole wall collapse
  in dry sand, with pre-water and re-bore in the planting head; auger commands are queued
- robot.launch.py runs the autonomy stack on hardware; GNSS receiver passthrough; shared
  config/robots.yaml; generated hardware interface contract
- Dockerfile (robot, sim, test), compose, systemd unit, CI, deployment and commissioning guide

Co-Authored-By: Claude Opus 5.5 <noreply@anthropic.com>

File: ros2_ws/src/fs_description/urdf/common.xacro (robot description, xacro)
@@ -48,9 +48,10 @@
   <!-- A wheel spinning about its local +y axis. shape: cylinder | sphere (sphere rides rough terrain better).
        With robot:=<name> the visual is that robot's CAD mesh for this link. -->
-  <xacro:macro name="wheel" params="name parent xyz r w m rim:=fs_yellow shape:=cylinder robot:=''">
+  <!-- effort: the most torque the drive can put on the wheel, N m (free-rolling wheels: bearing drag only) -->
+  <xacro:macro name="wheel" params="name parent xyz r w m rim:=fs_yellow shape:=cylinder robot:='' effort:=6000">
     <joint name="${name}_joint" type="continuous">
       <parent link="${parent}"/><child link="${name}_link"/>
       <origin xyz="${xyz}"/><axis xyz="0 1 0"/>
-      <limit effort="6000" velocity="40"/><dynamics damping="0.5"/>
+      <limit effort="${effort}" velocity="40"/><dynamics damping="0.5"/>
     </joint>
     <link name="${name}_link">
@@ -139,5 +140,5 @@
   <!-- Auger head: prismatic feed (positive = down along the tool), spin joint, auger link whose
        origin is at the feed carrier; the bit tip is at feed_axis * length. -->
-  <xacro:macro name="auger_head" params="robot parent xyz rpy:='0 0 0' length stroke feed_axis:='0 0 -1' spin_axis:='0 0 1'">
+  <xacro:macro name="auger_head" params="robot parent xyz rpy:='0 0 0' length stroke feed_axis:='0 0 -1' spin_axis:='0 0 1' mesh:='auger_link'">
     <joint name="auger_feed_joint" type="prismatic">
       <parent link="${parent}"/><child link="auger_feed_link"/>
@@ -155,5 +156,5 @@
     <link name="auger_link">
       <inertial><mass value="10"/><inertia ixx="0.3" iyy="0.3" izz="0.3" ixy="0" ixz="0" iyz="0"/></inertial>
-      <xacro:mesh_visual robot="${robot}" link="auger_link"/>
+      <xacro:mesh_visual robot="${robot}" link="${mesh}"/>
     </link>
   </xacro:macro>

File: ros2_ws/src/fs_description/urdf/jaal.urdf.xacro (robot description, xacro)
@@ -35,5 +35,5 @@
       <xacro:mesh_visual robot="${R}" link="steer_${tag}_link"/>
     </link>
-    <xacro:wheel name="wheel_${tag}" parent="steer_${tag}_link" xyz="0 0 -0.25" r="0.38" w="0.22" m="35" robot="${R}"/>
+    <xacro:wheel effort="900" name="wheel_${tag}" parent="steer_${tag}_link" xyz="0 0 -0.25" r="0.38" w="0.22" m="35" robot="${R}"/>
   </xacro:macro>
   <xacro:module tag="fl" x="0.95" y="0.83"/>

File: ros2_ws/src/fs_description/urdf/katar.urdf.xacro (robot description, xacro)
@@ -16,7 +16,11 @@
   <xacro:arg name="gnss_sigma" default="0.02"/>
   <xacro:arg name="inspect_cam" default="false"/>
-  <!-- feed stroke of the auger: 1.3 m bores ~0.55 m below grade; the deep-auger kit (2.0 m) bores the
-       1.2 m CSSRI auger holes through a kankar pan on sodic land -->
-  <xacro:arg name="auger_stroke" default="1.3"/>
+  <!-- deep-auger kit for the 1.2 m CSSRI auger holes through a kankar pan: a 1.45 m auger on a 1.5 m feed
+       (the standard 0.95 m auger on 1.3 m bores ~0.55 m below grade). The motor carriage stays above
+       ground either way: it rides the turret's feed mast. -->
+  <xacro:arg name="deep_auger" default="false"/>
+  <xacro:property name="deep" value="${'$(arg deep_auger)' in ('true', 'True', '1')}"/>
+  <xacro:property name="auger_len" value="${1.45 if deep else 0.95}"/>
+  <xacro:property name="auger_stroke" value="${1.5 if deep else 1.3}"/>
   <xacro:property name="ns" value="$(arg ns)"/>
   <xacro:property name="R" value="katar"/>
@@ -29,6 +33,6 @@
   </link>
   <xacro:person parent="base_link" name="driver" xyz="-0.12 0 0.44" robot="${R}"/>
-  <xacro:wheel name="rear_left_wheel" parent="base_link" xyz="0 0.8 0" r="0.72" w="0.4" m="120" robot="${R}"/>
-  <xacro:wheel name="rear_right_wheel" parent="base_link" xyz="0 -0.8 0" r="0.72" w="0.4" m="120" robot="${R}"/>
+  <xacro:wheel effort="7000" name="rear_left_wheel" parent="base_link" xyz="0 0.8 0" r="0.72" w="0.4" m="120" robot="${R}"/>
+  <xacro:wheel effort="7000" name="rear_right_wheel" parent="base_link" xyz="0 -0.8 0" r="0.72" w="0.4" m="120" robot="${R}"/>
   <xacro:macro name="steered_front" params="side y">
     <joint name="front_${side}_steer_joint" type="revolute">
@@ -41,5 +45,5 @@
       <xacro:mesh_visual robot="${R}" link="front_${side}_steer_link"/>
     </link>
-    <xacro:wheel name="front_${side}_wheel" parent="front_${side}_steer_link" xyz="0 0 0" r="0.42" w="0.24" m="40" robot="${R}"/>
+    <xacro:wheel effort="50" name="front_${side}_wheel" parent="front_${side}_steer_link" xyz="0 0 0" r="0.42" w="0.24" m="40" robot="${R}"/>
   </xacro:macro>
   <xacro:steered_front side="left" y="0.68"/>
@@ -61,8 +65,8 @@
   </link>
   <xacro:person parent="trailer_link" name="loader" xyz="-3.1 0 0.43" rpy="0 0 ${PI/2}" robot="${R}"/>
-  <xacro:wheel name="trailer_fl_wheel" parent="trailer_link" xyz="-3.1 0.93 -0.08" r="0.42" w="0.26" m="30" robot="${R}"/>
-  <xacro:wheel name="trailer_fr_wheel" parent="trailer_link" xyz="-3.1 -0.93 -0.08" r="0.42" w="0.26" m="30" robot="${R}"/>
-  <xacro:wheel name="trailer_rl_wheel" parent="trailer_link" xyz="-3.95 0.93 -0.08" r="0.42" w="0.26" m="30" robot="${R}"/>
-  <xacro:wheel name="trailer_rr_wheel" parent="trailer_link" xyz="-3.95 -0.93 -0.08" r="0.42" w="0.26" m="30" robot="${R}"/>
+  <xacro:wheel effort="50" name="trailer_fl_wheel" parent="trailer_link" xyz="-3.1 0.93 -0.08" r="0.42" w="0.26" m="30" robot="${R}"/>
+  <xacro:wheel effort="50" name="trailer_fr_wheel" parent="trailer_link" xyz="-3.1 -0.93 -0.08" r="0.42" w="0.26" m="30" robot="${R}"/>
+  <xacro:wheel effort="50" name="trailer_rl_wheel" parent="trailer_link" xyz="-3.95 0.93 -0.08" r="0.42" w="0.26" m="30" robot="${R}"/>
+  <xacro:wheel effort="50" name="trailer_rr_wheel" parent="trailer_link" xyz="-3.95 -0.93 -0.08" r="0.42" w="0.26" m="30" robot="${R}"/>
   <!-- ===================== boom ===================== -->
   <joint name="sled_joint" type="prismatic">
@@ -101,5 +105,6 @@
     <xacro:mesh_visual robot="${R}" link="turret_link"/>
   </link>
-  <xacro:auger_head robot="${R}" parent="turret_link" xyz="0.2 0 -0.06" length="0.95" stroke="$(arg auger_stroke)"/>
+  <xacro:auger_head robot="${R}" parent="turret_link" xyz="0.2 0 -0.06" length="${auger_len}" stroke="${auger_stroke}"
+                    mesh="${'auger_link_deep' if deep else 'auger_link'}"/>
   <xacro:duckbill_head robot="${R}" parent="turret_link" xyz="-0.2 0 -0.06" stroke="1.6" tamp_xyz="-0.2 0 -0.20" tamp_stroke="1.6"/>
   <!-- boom-side lidar, 0.3 m above ground, watching the strip the boom works in -->
@@ -150,7 +155,7 @@
       <soil_map>$(arg soil_map)</soil_map>
       <feed_joint>auger_feed_joint</feed_joint><spin_joint>auger_spin_joint</spin_joint>
-      <tip_link>auger_link</tip_link><reaction_link>turret_link</reaction_link><tip_offset>0 0 -0.95</tip_offset><tool_axis>0 0 -1</tool_axis>
+      <tip_link>auger_link</tip_link><reaction_link>turret_link</reaction_link><tip_offset>0 0 -${auger_len}</tip_offset><tool_axis>0 0 -1</tool_axis>
       <diameter>0.15</diameter><max_power>8000</max_power><efficiency>0.75</efficiency>
-      <max_thrust>8000</max_thrust><max_feed>0.15</max_feed><rpm>90</rpm><max_stroke>$(arg auger_stroke)</max_stroke>
+      <max_thrust>8000</max_thrust><max_feed>0.15</max_feed><rpm>90</rpm><max_stroke>${auger_stroke}</max_stroke>
       <free_speed>0.5</free_speed><retract_speed>0.6</retract_speed>
       <cmd_topic>/model/${ns}/auger/cmd</cmd_topic><status_topic>/model/${ns}/auger/status</status_topic>

File: ros2_ws/src/fs_description/urdf/pahadi.urdf.xacro (robot description, xacro)
@@ -27,10 +27,10 @@
     <xacro:mesh_visual robot="${R}" link="base_link"/>
   </link>
-  <xacro:wheel robot="${R}" name="fl1" parent="base_link" xyz="0.4 0.5 0" r="${WR}" w="0.28" m="12" shape="sphere" rim="fs_steel"/>
-  <xacro:wheel robot="${R}" name="fl2" parent="base_link" xyz="0.0 0.5 0" r="${WR}" w="0.28" m="12" shape="sphere" rim="fs_steel"/>
-  <xacro:wheel robot="${R}" name="fl3" parent="base_link" xyz="-0.4 0.5 0" r="${WR}" w="0.28" m="12" shape="sphere" rim="fs_steel"/>
-  <xacro:wheel robot="${R}" name="fr1" parent="base_link" xyz="0.4 -0.5 0" r="${WR}" w="0.28" m="12" shape="sphere" rim="fs_steel"/>
-  <xacro:wheel robot="${R}" name="fr2" parent="base_link" xyz="0.0 -0.5 0" r="${WR}" w="0.28" m="12" shape="sphere" rim="fs_steel"/>
-  <xacro:wheel robot="${R}" name="fr3" parent="base_link" xyz="-0.4 -0.5 0" r="${WR}" w="0.28" m="12" shape="sphere" rim="fs_steel"/>
+  <xacro:wheel effort="250" robot="${R}" name="fl1" parent="base_link" xyz="0.4 0.5 0" r="${WR}" w="0.28" m="12" shape="sphere" rim="fs_steel"/>
+  <xacro:wheel effort="250" robot="${R}" name="fl2" parent="base_link" xyz="0.0 0.5 0" r="${WR}" w="0.28" m="12" shape="sphere" rim="fs_steel"/>
+  <xacro:wheel effort="250" robot="${R}" name="fl3" parent="base_link" xyz="-0.4 0.5 0" r="${WR}" w="0.28" m="12" shape="sphere" rim="fs_steel"/>
+  <xacro:wheel effort="250" robot="${R}" name="fr1" parent="base_link" xyz="0.4 -0.5 0" r="${WR}" w="0.28" m="12" shape="sphere" rim="fs_steel"/>
+  <xacro:wheel effort="250" robot="${R}" name="fr2" parent="base_link" xyz="0.0 -0.5 0" r="${WR}" w="0.28" m="12" shape="sphere" rim="fs_steel"/>
+  <xacro:wheel effort="250" robot="${R}" name="fr3" parent="base_link" xyz="-0.4 -0.5 0" r="${WR}" w="0.28" m="12" shape="sphere" rim="fs_steel"/>
   <!-- ===================== articulation (steered: +-30 deg yaw, passive +-15 deg roll) ===================== -->
   <joint name="artic_yaw_joint" type="revolute">
@@ -55,10 +55,10 @@
     <xacro:mesh_visual robot="${R}" link="rear_link"/>
   </link>
-  <xacro:wheel robot="${R}" name="rl1" parent="rear_link" xyz="-0.45 0.5 -0.25" r="${WR}" w="0.28" m="12" shape="sphere" rim="fs_steel"/>
-  <xacro:wheel robot="${R}" name="rl2" parent="rear_link" xyz="-0.85 0.5 -0.25" r="${WR}" w="0.28" m="12" shape="sphere" rim="fs_steel"/>
-  <xacro:wheel robot="${R}" name="rl3" parent="rear_link" xyz="-1.25 0.5 -0.25" r="${WR}" w="0.28" m="12" shape="sphere" rim="fs_steel"/>
-  <xacro:wheel robot="${R}" name="rr1" parent="rear_link" xyz="-0.45 -0.5 -0.25" r="${WR}" w="0.28" m="12" shape="sphere" rim="fs_steel"/>
-  <xacro:wheel robot="${R}" name="rr2" parent="rear_link" xyz="-0.85 -0.5 -0.25" r="${WR}" w="0.28" m="12" shape="sphere" rim="fs_steel"/>
-  <xacro:wheel robot="${R}" name="rr3" parent="rear_link" xyz="-1.25 -0.5 -0.25" r="${WR}" w="0.28" m="12" shape="sphere" rim="fs_steel"/>
+  <xacro:wheel effort="250" robot="${R}" name="rl1" parent="rear_link" xyz="-0.45 0.5 -0.25" r="${WR}" w="0.28" m="12" shape="sphere" rim="fs_steel"/>
+  <xacro:wheel effort="250" robot="${R}" name="rl2" parent="rear_link" xyz="-0.85 0.5 -0.25" r="${WR}" w="0.28" m="12" shape="sphere" rim="fs_steel"/>
+  <xacro:wheel effort="250" robot="${R}" name="rl3" parent="rear_link" xyz="-1.25 0.5 -0.25" r="${WR}" w="0.28" m="12" shape="sphere" rim="fs_steel"/>
+  <xacro:wheel effort="250" robot="${R}" name="rr1" parent="rear_link" xyz="-0.45 -0.5 -0.25" r="${WR}" w="0.28" m="12" shape="sphere" rim="fs_steel"/>
+  <xacro:wheel effort="250" robot="${R}" name="rr2" parent="rear_link" xyz="-0.85 -0.5 -0.25" r="${WR}" w="0.28" m="12" shape="sphere" rim="fs_steel"/>
+  <xacro:wheel effort="250" robot="${R}" name="rr3" parent="rear_link" xyz="-1.25 -0.5 -0.25" r="${WR}" w="0.28" m="12" shape="sphere" rim="fs_steel"/>
   <!-- ===================== 4-axis arm ===================== -->
   <joint name="arm_base_joint" type="fixed"><parent link="base_link"/><child link="arm_base_link"/><origin xyz="0.25 0 0.65"/></joint>
