Commit message: Add drivers, calibration, a certified safety layer and a survival model
- fs_hardware: CANopen CiA 402 drives under ros2_control, a mock bus,
  and nodes that serve the simulator's topics on a real machine
  (robot.launch.py hardware:=true).
- Calibration CLI: wheel scales, plate, shear ring, shear vane,
  drawbar pull and survival counts fit the models.
- Safety concept for the certified layer (PL d), scanner fields sized
  per ISO 13855, a PLC model in simulation, and a comfort layer that
  always stops before the protective field.
- Soil: moisture-dependent strength, a daily rain and drying model per
  region (date:=MM-DD), persistent multi-pass ruts, and dry-pit collapse
  with pre-water and re-bore.
- First-year seedling survival predicted for every planted spot.
- Jaal 0.32 m tyres, Pahadi 1.0 + 1.0 m arm; CAD rebuilt.
- Pahadi auger reaction moved to the wrist link so it bores again.
- Root inertia moved to a child link, removing the KDL warning.
- Browser lab uses the same soil model.

Co-Authored-By: Claude Opus 5.5 <noreply@anthropic.com>

File: ros2_ws/src/fs_description/urdf/jaal.urdf.xacro (robot description, xacro)
@@ -35,5 +35,5 @@
       <xacro:mesh_visual robot="${R}" link="steer_${tag}_link"/>
     </link>
-    <xacro:wheel effort="900" name="wheel_${tag}" parent="steer_${tag}_link" xyz="0 0 -0.25" r="0.38" w="0.22" m="35" robot="${R}"/>
+    <xacro:wheel effort="900" name="wheel_${tag}" parent="steer_${tag}_link" xyz="0 0 -0.25" r="0.38" w="0.32" m="42" robot="${R}"/>
   </xacro:macro>
   <xacro:module tag="fl" x="0.95" y="0.83"/>
@@ -145,8 +145,8 @@
       <soil_map>$(arg soil_map)</soil_map>
       <topic>/model/${ns}/terramechanics</topic>
-      <xacro:tm_wheel link="wheel_fl_link" r="0.38" b="0.22" l="0.19"/>
-      <xacro:tm_wheel link="wheel_fr_link" r="0.38" b="0.22" l="0.19"/>
-      <xacro:tm_wheel link="wheel_rl_link" r="0.38" b="0.22" l="0.19"/>
-      <xacro:tm_wheel link="wheel_rr_link" r="0.38" b="0.22" l="0.19"/>
+      <xacro:tm_wheel link="wheel_fl_link" r="0.38" b="0.32" l="0.19"/>
+      <xacro:tm_wheel link="wheel_fr_link" r="0.38" b="0.32" l="0.19"/>
+      <xacro:tm_wheel link="wheel_rl_link" r="0.38" b="0.32" l="0.19"/>
+      <xacro:tm_wheel link="wheel_rr_link" r="0.38" b="0.32" l="0.19"/>
     </plugin>
     <plugin filename="fs_auger_soil_system" name="fs::AugerSoil">

File: ros2_ws/src/fs_description/urdf/pahadi.urdf.xacro (robot description, xacro)
@@ -18,6 +18,6 @@
   <xacro:property name="R" value="pahadi"/>
   <xacro:arg name="inspect_cam" default="false"/>
-  <xacro:property name="L_UP" value="0.85"/>
-  <xacro:property name="L_FORE" value="0.85"/>
+  <xacro:property name="L_UP" value="1.0"/>
+  <xacro:property name="L_FORE" value="1.0"/>
   <xacro:include filename="$(find fs_description)/urdf/common.xacro"/>
   <!-- ===================== front module ===================== -->
@@ -175,5 +175,5 @@
       <soil_map>$(arg soil_map)</soil_map>
       <feed_joint>auger_feed_joint</feed_joint><spin_joint>auger_spin_joint</spin_joint>
-      <tip_link>auger_link</tip_link><tip_offset>0.36 0 0</tip_offset><tool_axis>1 0 0</tool_axis>
+      <tip_link>auger_link</tip_link><reaction_link>arm_wrist_link</reaction_link><tip_offset>0.36 0 0</tip_offset><tool_axis>1 0 0</tool_axis>
       <diameter>0.12</diameter><max_power>2000</max_power><efficiency>0.8</efficiency>
       <max_thrust>2500</max_thrust><max_feed>0.12</max_feed><rpm>110</rpm><max_stroke>0.45</max_stroke>
